File: kicad/d1_sensor_shield.kicad_sch (KiCad schematic)
At the start: 13 parts, among them U1 WeMos_D1_mini, U2 LM75B, U3 W25Q16JV

Commit message: Update SPI flash footprint, silkscreen
Parts:
- U3: footprint Package_SO:SOIC-8_3.9x4.9mm_P1.27mm -> Package_SO:SOIC-8_5.23x5.23mm_P1.27mm

Commit message: widen photocell footprint
Parts:
- R1, R2, R3: value 68 -> 1k5
- R4: footprint OptoDevice:R_LDR_4.9x4.2mm_P2.54mm_Vertical -> OptoDevice:R_LDR_5.1x4.3mm_P3.4mm_Vertical
Other:
- company: (none) -> Northeastern Wireless Club
Changed lines of the file:
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@@
     (date "2021-01-07")
     (rev "v0.1")
+    (company "Northeastern Wireless Club")
   )
   (junction (at 95.25 39.37) (diameter 1.016) (color 0 0 0 0))
@@
     (in_bom yes) (on_board yes)
     (property "Reference" "R1" (id 0) (at 83.82 25.4 90))
-    (property "Value" "68" (id 1) (at 83.82 27.813 90))
+    (property "Value" "1k5" (id 1) (at 83.82 27.813 90))
     (property "Footprint" "Resistor_SMD:R_1206_3216Metric_Pad1.30x1.75mm_HandSolder" (id 2) (at 83.82 30.48 0)
       (effects (font (size 1.27 1.27)) hide)
@@
     (in_bom yes) (on_board yes)
     (property "Reference" "R2" (id 0) (at 83.82 34.29 90))
-    (property "Value" "68" (id 1) (at 83.82 36.83 90))
+    (property "Value" "1k5" (id 1) (at 83.82 36.83 90))
     (property "Footprint" "Resistor_SMD:R_1206_3216Metric_Pad1.30x1.75mm_HandSolder" (id 2) (at 83.82 39.37 0)
       (effects (font (size 1.27 1.27)) hide)
@@
     (in_bom yes) (on_board yes)
     (property "Reference" "R3" (id 0) (at 83.82 43.18 90))
-    (property "Value" "68" (id 1) (at 83.82 45.72 90))
+    (property "Value" "1k5" (id 1) (at 83.82 45.72 90))
     (property "Footprint" "Resistor_SMD:R_1206_3216Metric_Pad1.30x1.75mm_HandSolder" (id 2) (at 83.82 48.26 0)
       (effects (font (size 1.27 1.27)) hide)
@@
       (effects (font (size 1.27 1.27)) (justify left))
     )
-    (property "Footprint" "OptoDevice:R_LDR_4.9x4.2mm_P2.54mm_Vertical" (id 2) (at 124.46 39.37 90)
+    (property "Footprint" "OptoDevice:R_LDR_5.1x4.3mm_P3.4mm_Vertical" (id 2) (at 124.46 39.37 90)
       (effects (font (size 1.27 1.27)) (justify left) hide)
     )
@@
     )
     (path "/00000000-0000-0000-0000-00005ff93446"
-      (reference "R1") (unit 1) (value "68") (footprint "Resistor_SMD:R_1206_3216Metric_Pad1.30x1.75mm_HandSolder")
+      (reference "R1") (unit 1) (value "1k5") (footprint "Resistor_SMD:R_1206_3216Metric_Pad1.30x1.75mm_HandSolder")
     )
     (path "/00000000-0000-0000-0000-00005ff93906"
-      (reference "R2") (unit 1) (value "68") (footprint "Resistor_SMD:R_1206_3216Metric_Pad1.30x1.75mm_HandSolder")
+      (reference "R2") (unit 1) (value "1k5") (footprint "Resistor_SMD:R_1206_3216Metric_Pad1.30x1.75mm_HandSolder")
     )
     (path "/00000000-0000-0000-0000-00005ff93b2e"
-      (reference "R3") (unit 1) (value "68") (footprint "Resistor_SMD:R_1206_3216Metric_Pad1.30x1.75mm_HandSolder")
+      (reference "R3") (unit 1) (value "1k5") (footprint "Resistor_SMD:R_1206_3216Metric_Pad1.30x1.75mm_HandSolder")
     )
     (path "/6d0ea08a-9bbc-4891-92fd-bdbedc951610"
-      (reference "R4") (unit 1) (value "R_Photo") (footprint "OptoDevice:R_LDR_4.9x4.2mm_P2.54mm_Vertical")
+      (reference "R4") (unit 1) (value "R_Photo") (footprint "OptoDevice:R_LDR_5.1x4.3mm_P3.4mm_Vertical")
     )
     (path "/00000000-0000-0000-0000-00005ffd2c8a"
